File: Hardware/AntennaModule/Front-End.kicad_sch (KiCad schematic)
At the start: 30 parts, among them U1 C0727J5003AHF-1, U2 C0727J5003AHF-1, U3 NJG1155UX2, U4 NT1192FAAE1S, U5 PD0922J5050S2HF, U6 NT1192FAAE1S, X1 TA1985A, X2 TE0133B

Commit message: スタックアップを決定
Connections:
- net +3.3VA: no longer C3.1, U3.2 (VDD), U3.6 (VCTL)
- new net +3.3VP: C3.1, U3.2 (VDD), U3.6 (VCTL)
Changed lines of the file:
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@@
 	)
 	(junction
+		(at 129.54 86.36)
+		(diameter 0)
+		(color 0 0 0 0)
+	)
+	(junction
 		(at 66.04 119.38)
 		(diameter 0)
@@
 	)
 	(junction
-		(at 129.54 86.36)
-		(diameter 0)
-		(color 0 0 0 0)
-	)
-	(junction
 		(at 170.18 121.92)
 		(diameter 0)
@@
 	)
 	(symbol
-		(lib_id "power:+3.3VA")
-		(at 129.54 68.58 0)
+		(lib_id "power:GND")
+		(at 142.24 73.66 0)
 		(unit 1)
 		(exclude_from_sim no)
@@
 		(on_board yes)
 		(dnp no)
-		(property "Reference" "#PWR08"
-			(at 129.54 72.39 0)
+		(property "Reference" "#PWR011"
+			(at 142.24 80.01 0)
 			(effects
 				(font
@@
 			)
 		)
-		(property "Value" "+3.3VA"
-			(at 129.54 64.77 0)
+		(property "Value" "GND"
+			(at 142.24 77.47 0)
 			(effects
 				(font
@@
 		)
 		(property "Footprint" ""
-			(at 129.54 68.58 0)
+			(at 142.24 73.66 0)
 			(effects
 				(font
@@
 		)
 		(property "Datasheet" ""
-			(at 129.54 68.58 0)
+			(at 142.24 73.66 0)
 			(effects
 				(font
@@
 			)
 		)
-		(property "Description" "Power symbol creates a global label with name \"+3.3VA\""
-			(at 129.54 68.58 0)
+		(property "Description" "Power symbol creates a global label with name \"GND\" , ground"
+			(at 142.24 73.66 0)
 			(effects
 				(font
@@
 			(project "AntennaModule"
 				(path "/6fea4726-6625-4d37-9d0c-c1a5d08d59ce/6a1a8a49-81e8-4900-a7b3-937741017566"
-					(reference "#PWR08")
+					(reference "#PWR011")
 					(unit 1)
 				)
@@
 	(symbol
 		(lib_id "power:GND")
-		(at 142.24 73.66 0)
+		(at 55.88 121.92 0)
 		(unit 1)
 		(exclude_from_sim no)
@@
 		(on_board yes)
 		(dnp no)
-		(property "Reference" "#PWR011"
-			(at 142.24 80.01 0)
+		(property "Reference" "#PWR031"
+			(at 55.88 128.27 0)
 			(effects
 				(font
@@
 		)
 		(property "Value" "GND"
-			(at 142.24 77.47 0)
+			(at 55.88 125.73 0)
 			(effects
 				(font
@@
 		)
 		(property "Footprint" ""
-			(at 142.24 73.66 0)
+			(at 55.88 121.92 0)
 			(effects
 				(font
@@
 		)
 		(property "Datasheet" ""
-			(at 142.24 73.66 0)
+			(at 55.88 121.92 0)
 			(effects
 				(font
@@
 		)
 		(property "Description" "Power symbol creates a global label with name \"GND\" , ground"
-			(at 142.24 73.66 0)
+			(at 55.88 121.92 0)
 			(effects
 				(font
@@
 			(project "AntennaModule"
 				(path "/6fea4726-6625-4d37-9d0c-c1a5d08d59ce/6a1a8a49-81e8-4900-a7b3-937741017566"
-					(reference "#PWR011")
+					(reference "#PWR031")
 					(unit 1)
 				)
@@
 	)
 	(symbol
-		(lib_id "power:GND")
-		(at 55.88 121.92 0)
+		(lib_id "Device:C_Small")
+		(at 73.66 93.98 90)
+		(mirror x)
 		(unit 1)
 		(exclude_from_sim no)
@@
 		(on_board yes)
 		(dnp no)
-		(property "Reference" "#PWR031"
-			(at 55.88 128.27 0)
+		(property "Reference" "C2"
+			(at 73.66 96.52 90)
 			(effects
 				(font
 					(size 1.27 1.27)
 				)
-				(hide yes)
 			)
 		)
-		(property "Value" "GND"
-			(at 55.88 125.73 0)
+		(property "Value" "4.7p"
+			(at 73.66 91.44 90)
 			(effects
 				(font
@@
 			)
 		)
-		(property "Footprint" ""
-			(at 55.88 121.92 0)
+		(property "Footprint" "Capacitor_SMD_extlib:C_Murata_xxx15_0402_1005Metric_1.0x0.5mm"
+			(at 73.66 93.98 0)
 			(effects
 				(font
@@
 			)
 		)
-		(property "Datasheet" ""
-			(at 55.88 121.92 0)
+		(property "Datasheet" "~"
+			(at 73.66 93.98 0)
 			(effects
 				(font
@@
 			)
 		)
-		(property "Description" "Power symbol creates a global label with name \"GND\" , ground"
-			(at 55.88 121.92 0)
+		(property "Description" "Unpolarized capacitor, small symbol"
+			(at 73.66 93.98 0)
 			(effects
 				(font
@@
 			)
 		)
+		(pin "2"
+		)
 		(pin "1"
 		)
@@
 			(project "AntennaModule"
 				(path "/6fea4726-6625-4d37-9d0c-c1a5d08d59ce/6a1a8a49-81e8-4900-a7b3-937741017566"
-					(reference "#PWR031")
+					(reference "C2")
 					(unit 1)
 				)
@@
 	)
 	(symbol
-		(lib_id "Device:C_Small")
-		(at 73.66 93.98 90)
-		(mirror x)
+		(lib_id "power:+3.3VP")
+		(at 129.54 86.36 0)
 		(unit 1)
 		(exclude_from_sim no)
@@
 		(on_board yes)
 		(dnp no)
-		(property "Reference" "C2"
-			(at 73.66 96.52 90)
+		(property "Reference" "#PWR041"
+			(at 133.35 87.63 0)
 			(effects
 				(font
 					(size 1.27 1.27)
 				)
+				(hide yes)
 			)
 		)
-		(property "Value" "4.7p"
-			(at 73.66 91.44 90)
+		(property "Value" "+3.3VP"
+			(at 129.54 82.55 0)
 			(effects
 				(font
@@
 			)
 		)
-		(property "Footprint" "Capacitor_SMD_extlib:C_Murata_xxx15_0402_1005Metric_1.0x0.5mm"
-			(at 73.66 93.98 0)
+		(property "Footprint" ""
+			(at 129.54 86.36 0)
 			(effects
 				(font
@@
 			)
 		)
-		(property "Datasheet" "~"
-			(at 73.66 93.98 0)
+		(property "Datasheet" ""
+			(at 129.54 86.36 0)
 			(effects
 				(font
@@
 			)
 		)
-		(property "Description" "Unpolarized capacitor, small symbol"
-			(at 73.66 93.98 0)
+		(property "Description" "Power symbol creates a global label with name \"+3.3VP\""
+			(at 129.54 86.36 0)
 			(effects
 				(font
@@
 			)
 		)
-		(pin "2"
-		)
 		(pin "1"
 		)
 		(instances
-			(project "AntennaModule"
+			(project ""
 				(path "/6fea4726-6625-4d37-9d0c-c1a5d08d59ce/6a1a8a49-81e8-4900-a7b3-937741017566"
-					(reference "C2")
+					(reference "#PWR041")
 					(unit 1)
 				)
@@
 	)
 	(symbol
+		(lib_id "power:+3.3VP")
+		(at 129.54 68.58 0)
+		(unit 1)
+		(exclude_from_sim no)
+		(in_bom yes)
+		(on_board yes)
+		(dnp no)
+		(property "Reference" "#PWR07"
+			(at 133.35 69.85 0)
+			(effects
+				(font
+					(size 1.27 1.27)
+				)
+				(hide yes)
+			)
+		)
+		(property "Value" "+3.3VP"
+			(at 129.54 64.77 0)
+			(effects
+				(font
+					(size 1.27 1.27)
+				)
+			)
+		)
+		(property "Footprint" ""
+			(at 129.54 68.58 0)
+			(effects
+				(font
+					(size 1.27 1.27)
+				)
+				(hide yes)
+			)
+		)
+		(property "Datasheet" ""
+			(at 129.54 68.58 0)
+			(effects
+				(font
+					(size 1.27 1.27)
+				)
+				(hide yes)
+			)
+		)
+		(property "Description" "Power symbol creates a global label with name \"+3.3VP\""
+			(at 129.54 68.58 0)
+			(effects
+				(font
+					(size 1.27 1.27)
+				)
+				(hide yes)
+			)
+		)
+		(pin "1"
+		)
+		(instances
+			(project "AntennaModule"
+				(path "/6fea4726-6625-4d37-9d0c-c1a5d08d59ce/6a1a8a49-81e8-4900-a7b3-937741017566"
+					(reference "#PWR07")
+					(unit 1)
+				)
+			)
+		)
+	)
+	(symbol
 		(lib_id "Device:C_Small")
 		(at 73.66 88.9 90)
@@
 					(unit 1)
 				)
-			)
-		)
-	)
-	(symbol
-		(lib_id "power:+3.3VA")
-		(at 129.54 86.36 0)
-		(unit 1)
-		(exclude_from_sim no)
-		(in_bom yes)
-		(on_board yes)
-		(dnp no)
-		(property "Reference" "#PWR07"
-			(at 129.54 90.17 0)
-			(effects
-				(font
-					(size 1.27 1.27)
-				)
-				(hide yes)
-			)
-		)
-		(property "Value" "+3.3VA"
-			(at 129.54 82.55 0)
-			(effects
-				(font
-					(size 1.27 1.27)
-				)
-			)
-		)
-		(property "Footprint" ""
-			(at 129.54 86.36 0)
-			(effects
-				(font
-					(size 1.27 1.27)
-				)
-				(hide yes)
-			)
-		)
-		(property "Datasheet" ""
-			(at 129.54 86.36 0)
-			(effects
-				(font
-					(size 1.27 1.27)
-				)
-				(hide yes)
-			)
-		)
-		(property "Description" "Power symbol creates a global label with name \"+3.3VA\""
-			(at 129.54 86.36 0)
-			(effects
-				(font
-					(size 1.27 1.27)
-				)
-				(hide yes)
-			)
-		)
-		(pin "1"
-		)
-		(instances
-			(project ""
-				(path "/6fea4726-6625-4d37-9d0c-c1a5d08d59ce/6a1a8a49-81e8-4900-a7b3-937741017566"
-					(reference "#PWR07")
-					(unit 1)
-				)
