File: Hardware/Antenna_Module/Antenna_Module.kicad_sch (KiCad schematic)
At the start: 18 parts, among them J1 Conn_Coaxial, J2 Conn_01x02_Pin, U1 C0727J5003AHF-1, U2 C0727J5003AHF-1, U3 TFM.120A

Commit message: データシート整理
Other:
- note added: "入力マッチング回路省略"
- note added: "出力マッチング回路省略"
- note removed: "入力マッチング回路略"
- note removed: "出力マッチング回路略"
- moved on the sheet: AE1A, AE1B, C1, C2, C3, C4, D1, D2, D3, D4, D5, D6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

Commit message: 基板設定済み
Parts:
- removed U1, U2: C0727J5003AHF-1, RF_Converter_extlib:Xinger_0805_2012Metric-6_Pad0.33x0.35mm, symbol RF_Converter_extlib:C0727J5003AHF-1
- added U1, U2: X3C14P1-03S-1, RF_Converter_extlib:RF_HybridCoupler_TTM_X3C14P1-03S, symbol RF_Converter_extlib:X3C14P1-03S-1
Connections:
- net GND: now also U1.5 (GND), U2.5 (GND)
- net at R1.1: now also U1.2 (Isolated)
- net at U3.2 (HB_IN): now also U1.1 (Input)
- net at C2.2: now also U1.4 (∠θ)
- net at C1.2: now also U1.3 (∠θ-90)
- net at AE1.3 (LB1), D4.2 (A2): now also U2.3 (∠θ-90)
- net at R2.1: now also U2.2 (Isolated)
- net at U3.35 (LB_IN): now also U2.1 (Input)
- net at AE1.4 (LB2), D2.1 (A1): now also U2.4 (∠θ)
