File: Hardware/Antenna_Module/Antenna_Module.kicad_pcb (KiCad board)
At the start: 4 copper layers, 80 x 80 mm, 54 parts, among them J1 Conn_01x10, SW1 ColdStart, U1 C0727J5003AHF-1, U2 C0727J5003AHF-1, U3 NJG1155UX2, U4 NT1192FAAE1S, U5 PD0922J5050S2HF, U6 NT1192FAAE1S, U7 NEO-D9C, U8 NEO-F9P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

Commit message: データシート整理
Parts:
- removed BT1: MS421R, Battery_extlib:Battery_Seiko_MS421R
- removed C10: 2.2u, Capacitor_SMD:C_0603_1608Metric
- removed C11, C9: 1u, Capacitor_SMD:C_0603_1608Metric
- removed C5: 2.4p, Capacitor_SMD_extlib:C_Murata_xxx15_0402_1005Metric_1.0x0.5mm
- removed C6: 1000p, Capacitor_SMD_extlib:C_Murata_xxx15_0402_1005Metric_1.0x0.5mm
- removed C7, C8: 1p, Capacitor_SMD_extlib:C_Murata_xxx15_0402_1005Metric_1.0x0.5mm
- removed L1: 12nH, Inductor_SMD_extlib:L_Murata_LQW15ANxxxx80x_0402_1005Metric_1.0x0.6mm
- removed L2, L6: 20nH, Inductor_SMD_extlib:L_Murata_LQW15ANxxxx80x_0402_1005Metric_1.0x0.6mm
- removed L3: 3.3nH, Inductor_SMD_extlib:L_Murata_LQW15ANxxxx80x_0402_1005Metric_1.0x0.6mm
- removed L4: 5.6nH, Inductor_SMD_extlib:L_Murata_LQW15ANxxxx80x_0402_1005Metric_1.0x0.6mm
- removed L5: 3.6nH, Inductor_SMD_extlib:L_Murata_LQW15ANxxxx80x_0402_1005Metric_1.0x0.6mm
- removed R10, R4, R5, R6, R7, R9: 33, Resistor_SMD:R_0402_1005Metric
- removed R11: 1k, Resistor_SMD:R_0402_1005Metric
- removed R3: 100, Resistor_SMD_extlib:R_Vishay_FC0603xxxxxxTxx_0603_1608Metric_1.626x0.813mm
- removed R8: 3.3k, Resistor_SMD:R_0402_1005Metric
- removed REF**: Taoglas_TFM.120A_GNSS, RF_FEM_extlib:Taoglas_TFM.120A_GNSS
- removed SW1: ColdStart, Button_Switch_SMD:SW_Push_1P1T_NO_Vertical_Wuerth_434133025816
- removed TP1: ~{SAFEBOOT_F9P}, TestPoint:TestPoint_Pad_D1.0mm
- removed TP2: ~{SAFEBOOT_D9C}, TestPoint:TestPoint_Pad_D1.0mm
- removed TP3: EXTINT_F9P, TestPoint:TestPoint_Pad_D1.0mm
- removed TP4: EXTINT_D9C, TestPoint:TestPoint_Pad_D1.0mm
- removed TP5: LNA_EN, TestPoint:TestPoint_Pad_D1.0mm
- removed U4, U6: NT1192FAAE1S, RF_LNA_extlib:Nisshinbo_EPFFP-6-FA
- removed U5: PD0922J5050S2HF, RF_Converter_extlib:Xinger_0805_2012Metric-6_Pad0.33x0.41mm
- removed U7: NEO-D9C, RF_GNSS_extlib:ublox_NEO
- removed U8: NEO-F9P, RF_GNSS_extlib:ublox_NEO
- removed X1: TA1985A, Filter_extlib:Filter_SAW-6_3.0x3.0mm
- removed X2: TE0133B, Filter_extlib:Filter_SAW-8_3.0x3.0mm
- added J2: Conn_01x02_Pin, Connector_PinHeader_2.54mm:PinHeader_1x02_P2.54mm_Vertical, F.Cu at (157.6, 133.0)
- AE1: moved to F.Cu
- C3: value 1000p -> 100p
- D1: value CUHS20S30 -> AXGD10402KR; footprint Diode_SMD_extlib:D_Toshiba_US2H -> Diode_SMD_extlib:D_Littelfuse_AXGD10402KR_0402_1005Metric_1.02x0.51mm
- D6: value PULSE -> AXGD10402KR; footprint LED_SMD:LED_0402_1005Metric -> Diode_SMD_extlib:D_Littelfuse_AXGD10402KR_0402_1005Metric_1.02x0.51mm
- J1: value Conn_01x10 -> Conn_Coaxial; footprint Connector_PinHeader_1.27mm:PinHeader_2x05_P1.27mm_Vertical_SMD -> Connector_Coaxial:U.FL_Hirose_U.FL-R-SMT-1_Vertical
- U3: value NJG1155UX2 -> TFM.120A; footprint RF_LNA_extlib:Nisshinbo_EPFFP-6-FA -> RF_FEM_extlib:Taoglas_TFM.120A_GNSS
- moved J1 160.1 mm to (40.8, 107.6), turned to 180 degrees
- moved D1 110.3 mm to (78.9, 120.3)
- moved D6 107.8 mm to (78.9, 133.0), turned to 0 degrees
- moved C3 98.8 mm to (78.9, 145.7), turned to 0 degrees
- moved C4 95.9 mm to (78.9, 148.3), turned to 0 degrees
- moved C1 89.1 mm to (78.9, 140.6), turned to 0 degrees
- moved R1 85.3 mm to (78.9, 135.6), turned to 0 degrees
- moved C2 84.1 mm to (78.9, 143.2), turned to 0 degrees
- moved D3 80.9 mm to (78.9, 125.4)
- moved D4 80.0 mm to (78.9, 127.9), turned to 0 degrees
- moved R2 76.8 mm to (78.9, 138.1), turned to 0 degrees
- moved AE1 75.0 mm to (150.0, 25.0), turned to 0 degrees
- moved D2 73.6 mm to (78.9, 122.9)
- moved U1 73.4 mm to (81.4, 115.2), turned to 0 degrees
- moved D5 68.5 mm to (78.9, 130.5), turned to 0 degrees
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Connections:
- C3 pad 1: +3.3VP -> +3.3V
- C4 pad 1: +3.3VA -> +3.3V
- D1 pad 1: Net-(D1-K) -> Net-(AE1A-HB2)
- D1 pad 2: +3.3V -> GND
- D2 pad 1: Net-(AE1A-HB2) -> Net-(AE1B-LB2)
- D4 pad 1: Net-(AE1B-LB2) -> GND
- D4 pad 2: GND -> Net-(AE1B-LB1)
- D5 pad 2: Net-(AE1B-LB1) -> +3.3V
- D6 pad 1: GNDD -> GND
- D6 pad 2: Net-(D6-A) -> Net-(D6-A2)
- J1 pad 1: GNDD -> Net-(D6-A2)
- J1 pad 2: +3.3V -> GND
- U3 pad 2: +3.3VP -> Net-(U1-Input)
- U3 pad 3: Net-(U3-RFOUT) -> GND
- U3 pad 5: Net-(U3-RFIN) -> GND
- U3 pad 6: +3.3VP -> GND
Routing:
- net Net-(U2-Input): track 20.1 -> 0.00 mm
- net Net-(U1-Input): track 16.0 -> 0.00 mm
- net +3.3VA: track 9.80 -> 0.00 mm
- net Net-(U5-Output1): track 7.99 -> 0.00 mm
- net /RF_IN_D9C: track 7.44 -> 0.00 mm
- net /RF_IN_F9P: track 4.73 -> 0.00 mm
- net Net-(AE1B-LB2): track 2.31 -> 0.00 mm
- net Net-(AE1B-LB1): track 2.31 -> 0.00 mm
- net Net-(U5-Output2): track 2.29 -> 0.00 mm
- net Net-(AE1A-HB2): track 2.21 -> 0.00 mm
- net Net-(AE1A-HB1): track 2.21 -> 0.00 mm
- net +3.3VP: track 2.04 -> 0.00 mm
- net Net-(U4-RFOUT): track 1.27 -> 0.00 mm
- net Net-(U3-RFOUT): track 1.02 -> 0.00 mm
- net GND: vias 288 -> 0
Other:
- board text removed: "↓ここは50Ωじゃなくてもいいので0.66mm"
- board text removed: "ここは50Ωなので0.605mm↗"
- board text removed: "曲げ半径は配線幅の3倍以上 抵抗の中心xは接続するパッドの中心xから外側に0.145オフセット 上カプラは25milグリッドから0.0025mm下にずれてる -(0.605-0.35)/2 カプラのパッドX位置から伝送線路X位置のオフセット RFINパッドの高さは25milグリッド揃え"
- board text removed: "電源リターンパス"

Commit message: 基板設定済み
Parts:
- AE1: moved to B.Cu
- U1, U2: value C0727J5003AHF-1 -> X3C14P1-03S-1; footprint RF_Converter_extlib:Xinger_0805_2012Metric-6_Pad0.33x0.35mm -> RF_Converter_extlib:RF_HybridCoupler_TTM_X3C14P1-03S
- moved J2 220.6 mm to (-30.5, 17.8)
- moved D6 189.8 mm to (-33.0, -20.3)
- moved U3 184.5 mm to (-25.4, 0.00)
- moved AE1 152.1 mm to (0.00, 0.00), turned to -45 degrees
- moved U1 151.7 mm to (0.00, -12.7)
- moved J1 145.2 mm to (-27.9, -20.3), turned to 0 degrees
- moved U2 134.5 mm to (0.00, 10.2), turned to 180 degrees
- moved C2 97.4 mm to (22.9, 63.5)
- moved C3 97.4 mm to (22.9, 66.0)
- moved C4 97.4 mm to (22.9, 68.6)
- moved D1 97.4 mm to (22.9, 40.6)
- moved D2 97.4 mm to (22.9, 43.2)
- moved D3 97.4 mm to (22.9, 45.7)
- moved D4 97.4 mm to (22.9, 48.3)
- moved D5 97.4 mm to (22.9, 50.8)
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Connections:
- U1 pad 2: GND -> Net-(U1-Isolated)
- U1 pad 3: Net-(U1-Isolated) -> Net-(U1-∠θ-90)
- U2 pad 2: GND -> Net-(U2-Isolated)
- U2 pad 3: Net-(U2-Isolated) -> Net-(AE1B-LB1)
Routing:
- removed copper zone on B.Cu, net GND
- removed copper zone on F.Cu, net GND
- removed copper zone on In1.Cu, net GND
- removed copper zone on In2.Cu, net GND
Other:
- copper layers 4 -> 2
- board text removed: "0"
- board text removed: "0 mm"
- board text removed: "0.01 mm"
- board text removed: "0.0152 mm"
- board text removed: "0.02"
- board text removed: "0.035 mm"
- board text removed: "0.1000 mm / 0.1000 mm"
- board text removed: "0.1164 mm"
- board text removed: "0.1500 mm"
- board text removed: "0.218 mm"
- board text removed: "0.4 mm"
- board text removed: "0.4mm H/HOZ without copper"
- board text removed: "1"
- board text removed: "1.6252 mm"
- board text removed: "2116 RC54% 4.9mil"
- board text removed: "3.8"
- board text removed: "4"
- board text removed: "4.4"
- board text removed: "4.6"
- board text removed: "7628, RC 49%, 8.6 mil"
- board text removed: "80.0025 mm x 80.0025 mm"
- board text removed: "B.Cu"
- board text removed: "B.Mask"
- board text removed: "B.Paste"
- board text removed: "B.Silkscreen"
- board text removed: "Bottom Silk Screen"
- board text removed: "Bottom Solder Mask"
- board text removed: "Bottom Solder Paste"
- board text removed: "ENIG"
- board text removed: "F.Cu"
- board text removed: "F.Mask"
- board text removed: "F.Paste"
- board text removed: "F.Silkscreen"
- board text removed: "In1.Cu"
- board text removed: "In2.Cu"
- board text removed: "JLC04161H-7628B"
- board text removed: "Not specified"
- board text removed: "Top Silk Screen"
- board text removed: "Top Solder Mask"
- board text removed: "Top Solder Paste"
- board text removed: "copper"
- board text removed: "core"
- board text removed: "prepreg"
- board text removed: "εR"
- board text removed: "いいえ"
- board text removed: "はい"
- board text removed: "インピーダンス制御:"
- board text removed: "エッジ カード コネクタ:"
- board text removed: "カラー"
- board text removed: "タイプ"
- board text removed: "レイヤー名"
- board text removed: "基板の特性"
- board text removed: "基板全体の寸法:"
- board text removed: "基板厚:"
- board text removed: "基板端メッキ:"
- board text removed: "導体レイヤー数:"
- board text removed: "損失正接"
- board text removed: "最小穴径:"
- board text removed: "最小配線幅/間隔:"
- board text removed: "材料"
- board text removed: "端面スルーホール パッド:"
- board text removed: "線幅 (mm)"
- board text removed: "誘電体 1 (1/3)"
- board text removed: "誘電体 2"
- board text removed: "誘電体 3 (1/3)"
- board text removed: "銅箔仕上げ:"

Commit message: 配線
Parts:
- moved R1 75.8 mm to (2.59, -17.2), turned to 90 degrees
- moved C2 75.4 mm to (-2.97, -7.32), turned to 75 degrees
- moved C1 71.1 mm to (2.97, -7.32), turned to 105 degrees
- moved D3 55.2 mm to (2.87, -5.72), turned to 15 degrees
- moved D1 53.0 mm to (-2.87, -5.72), turned to -15 degrees
- moved R2 50.2 mm to (-2.59, 15.1), turned to -90 degrees
- moved D4 49.8 mm to (-6.63, 8.15), turned to -90 degrees
- moved D2 38.6 mm to (6.63, 8.15), turned to 90 degrees
- moved C3 19.3 mm to (30.5, 48.3)
- moved C4 19.3 mm to (30.5, 50.8)
- moved U2 0.46 mm to (0.00, 10.6)
Routing:
- net Net-(AE1B-LB2): track 0.00 -> 6.07 mm
- net Net-(AE1B-LB1): track 0.00 -> 6.07 mm
- net Net-(U1-∠θ-90): track 0.00 -> 2.01 mm
- net Net-(U1-∠θ): track 0.00 -> 2.01 mm
- net GND: vias 0 -> 158
- added copper zone on B.Cu, net GND
- added copper zone on F.Cu, net GND

Commit message: ビア配置
Parts:
- moved C3 71.6 mm to (-33.0, 15.2)
- moved C4 70.6 mm to (-30.5, 15.2)
- moved D5 62.7 mm to (-30.5, 17.8)
- moved D6 5.48 mm to (-27.9, -22.4), turned to 90 degrees
- moved J1 3.59 mm to (-25.4, -22.9)
- moved J2 2.54 mm to (-30.5, 20.3)
- moved U3 1.27 mm to (-24.1, 0.00)
Routing:
- net Net-(U2-Input): track 0.00 -> 25.9 mm
- net Net-(U1-Input): track 0.00 -> 22.8 mm
- net GND: vias 158 -> 384
Other:
- board text added: "カプラ下は0.2mmビア"

Commit message: 配線
Parts:
- added REF**: KiCad-Logo2_5mm_SilkScreen, Symbol:KiCad-Logo2_5mm_SilkScreen, F.Cu at (0.00, -30.6)
- moved D6 5.08 mm to (-27.9, -17.3)
- moved J1 5.08 mm to (-25.4, -17.8)
- moved C4 3.38 mm to (-33.9, 15.4)
- moved C3 1.16 mm to (-33.9, 14.4)
- moved D5 0.48 mm to (-30.0, 17.8), turned to 180 degrees
Routing:
- net GND: vias 384 -> 394
Other:
- board text added: "3V3"
- board text added: "CelestNavi"
- board text added: "GND"
- board text added: "RFOUT"
- board text added: "星導"
